File: locator_beacon.kicad_sch (KiCad schematic)
At the start: 9 parts, among them J1 Conn_01x02, J3 Conn_01x01, J4 OSHW logo, J5 Conn_01x02, J6 Conn_01x01, J7 Conn_01x01, J8 Conn_01x01, U13 Pico

Commit message: 555 driver
Parts:
- removed D1: DSS16U, Diode_SMD:D_SOD-123, symbol Diode:B120-E3
- removed J1: Conn_01x02, custom:SAMTEC_TSM-102-01-L-SH, symbol custom_symbols:TSM-102-01-L-SH
- removed J3, J6, J7, J8: Conn_01x01, Connector_PinHeader_2.54mm:PinHeader_1x01_P2.54mm_Vertical, symbol Connector_Generic:Conn_01x01
- removed J5: Conn_01x02, Connector_PinHeader_2.54mm:PinHeader_1x02_P2.54mm_Vertical, symbol Connector_Generic:Conn_01x02
- removed U13: Pico, custom:RPi_pico, symbol MCU_RaspberryPi_and_Boards:Pico
- added BT1: Battery_Cell, Connector_PinHeader_2.54mm:PinHeader_1x02_P2.54mm_Vertical, symbol Device:Battery_Cell
- added C1, C3: 1.5n, Capacitor_SMD:C_0805_2012Metric, symbol Device:C
- added C10, C9: 220n, Capacitor_SMD:C_0805_2012Metric, symbol Device:C
- added C11, C13, C4, C5, C7: 10u, Capacitor_SMD:C_0805_2012Metric, symbol Device:C
- added C12: C, Capacitor_SMD:CP_Elec_4x3.9, symbol Device:C_Polarized
- added C14, C15: 1n, Capacitor_SMD:C_0805_2012Metric, symbol Device:C
- added C2: C, Capacitor_SMD:C_0805_2012Metric, symbol Device:C_Polarized
- added C6: 10u, Capacitor_SMD:CP_Elec_4x3.9, symbol Device:C_Polarized
- added C8: 10n, Capacitor_SMD:C_0805_2012Metric, symbol Device:C
- added D2, D3: DSS16U, Diode_SMD:D_SOD-123, symbol Diode:B120-E3
- added J1: Conn_01x02_Pin, Connector_PinSocket_1.27mm:PinSocket_1x02_P1.27mm_Vertical, symbol Connector:Conn_01x02_Pin
- added J2: Conn_01x02_Pin, Connector_PinHeader_1.27mm:PinHeader_1x02_P1.27mm_Vertical, symbol Connector:Conn_01x02_Pin
- added L1, L2: 10u, Capacitor_SMD:C_0805_2012Metric, symbol Device:L
- added OUT1: Speaker, Connector_PinSocket_2.54mm:PinSocket_1x02_P2.54mm_Vertical, symbol Device:Speaker
- added Q1, Q2, Q3, Q4: DMN6140L, Package_TO_SOT_SMD:SOT-23, symbol Transistor_FET:DMN6140L
- added R1, R11, R3, R5, R7, R9: 2k, Resistor_SMD:R_0805_2012Metric, symbol Device:R
- added R10, R12: 500, Resistor_SMD:R_0805_2012Metric, symbol Device:R
- added R13: 8.2k, Resistor_SMD:R_0805_2012Metric, symbol Device:R
- added R14: 68k, Resistor_SMD:R_0805_2012Metric, symbol Device:R
- added R15, R16: 100k, Resistor_SMD:R_0805_2012Metric, symbol Device:R
- added R2: 42.3k, Resistor_SMD:R_0805_2012Metric, symbol Device:R
- added R4: 5k, Resistor_SMD:R_0805_2012Metric, symbol Device:R
- added R6: 10k, Resistor_SMD:R_0805_2012Metric, symbol Device:R
- added R8: 100, Resistor_SMD:R_0805_2012Metric, symbol Device:R
- added RV1: 100k, Potentiometer_SMD:Potentiometer_Bourns_3314J_Vertical, symbol Device:R_Potentiometer_Trim
- added TP1: +12, TestPoint:TestPoint_Pad_D1.0mm, symbol Connector:TestPoint
- added TP2: LHI, TestPoint:TestPoint_Pad_D1.0mm, symbol Connector:TestPoint
- added TP3: HV, TestPoint:TestPoint_Pad_D1.0mm, symbol Connector:TestPoint
- added TP4: LLO, TestPoint:TestPoint_Pad_D1.0mm, symbol Connector:TestPoint
- added TP5: RHI, TestPoint:TestPoint_Pad_D1.0mm, symbol Connector:TestPoint
- added TP6: RLO, TestPoint:TestPoint_Pad_D1.0mm, symbol Connector:TestPoint
- added U1: MIC4606, Package_SO:TSSOP-16-1EP_4.4x5mm_P0.65mm, symbol custom_symbols:MIC4606
- added U2, U4: MIC2288, Package_SO:TSOP-5_1.65x3.05mm_P0.95mm, symbol custom_symbols:MIC2288
- added U3: LM556, Package_SO:SO-14_3.9x8.65mm_P1.27mm, symbol Timer:LM556
- added U5, U6: MIC7300, digikey-footprints:SOT-753, symbol Digikey:AD8605ARTZ-REEL7
- J4: footprint Symbol:OSHW-Logo_5.7x6mm_Copper -> Symbol:OSHW-Logo_5.7x6mm_SilkScreen
Connections:
- net +BATT: now also BT1.1 (+), C2.1, J1.1 (Pin_1), L2.1, U4.4 (EN), U4.5 (VIN)
- net GND: now also BT1.2 (-), C1.2, C10.2, C11.2, C12.2, C13.2, C14.2, C15.2, C2.2, C3.2, C4.2, C6.2, C8.2, C9.2, J1.2 (Pin_2), Q2.2 (S), Q4.2 (S), R16.2, R4.2, RV1.3, U1.13 (VSS), U2.2 (GND), U3.7 (GND), U3.7 (GND), U4.2 (GND), U5.2 (V-), U6.2 (V-)
- new net: R6.2, R8.1, U3.1 (DIS)
- new net: D2.2 (A), L2.2, U4.1 (SW)
- new net: R9.2, U1.9 (AHO)
- new net: D3.2 (A), L1.2, U2.1 (SW)
- new net: R3.1, U1.6 (APWM)
- new net: R7.2, U1.14 (BLO)
- new net: RV1.2, U2.3 (FB)
- new net: C8.1, U3.3 (CV)
- new net: C5.1, U1.1 (BHB)
- new net: R11.2, U1.11 (ALO)
- new net: R5.2, U1.16 (BHO)
- new net: R1.1, U1.3 (BPWM)
- new net: C7.1, U1.8 (AHB)
- new net: C15.1, R15.2, R16.1, U6.3
- new net: R2.2, R4.1, U4.3 (FB)
- new net: R10.2, R12.1, U5.3
- new net: R13.2, R14.1, U3.13 (DIS)
- new net: C13.1, R12.2
- new net: U3.11 (CV), U5.1, U5.4
- new net +12V: C4.1, C6.1, D2.1 (K), L1.1, R13.1, R15.1, R2.1, R6.1, TP1.1, U1.12 (VDD), U1.2 (EN), U2.4 (EN), U2.5 (VIN), U3.14 (VCC), U3.14 (VCC), U3.4 (R), U5.5 (V+), U6.5 (V+)
- new net A: C14.1, R14.2, U3.12 (THR), U3.8 (TR)
- new net B: C11.1, R8.2, U3.2 (THR), U3.6 (TR)
- new net HV: C12.1, D3.1 (K), Q1.3 (D), Q3.3 (D), RV1.1, TP3.1
- new net L_HI: Q1.1 (G), R5.1, TP2.1
- new net L_LO: Q2.1 (G), R7.1, TP4.1
- new net OUT_A: C5.2, C9.1, J2.2 (Pin_2), OUT1.2, Q1.2 (S), Q2.3 (D), U1.15 (BHS)
- new net OUT_B: C10.1, C7.2, J2.1 (Pin_1), OUT1.1, Q3.2 (S), Q4.3 (D), U1.10 (AHS)
- new net PULSE_START: R10.1, U3.10 (R), U3.5 (Q)
- new net PWM_A: C1.1, R3.2, U3.9 (Q), U6.4
- new net PWM_B: C3.1, R1.2, U6.1
- new net R_HI: Q3.1 (G), R9.1, TP5.1
- new net R_LO: Q4.1 (G), R11.1, TP6.1
Other:
- removed sheet amplifier
- removed sheet power
- note added: "+12 source"
- note added: "Battery"
- note added: "Chirp generator"
- note added: "Full bridge"
- note added: "Gate driver"
- note added: "HV source"
- note added: "Misc"
- note added: "Output filter"
- note added: "pulse control"

Commit message: Work
Parts:
- removed R14: 68k, Resistor_SMD:R_0805_2012Metric, symbol Device:R
- removed R15, R16: 100k, Resistor_SMD:R_0805_2012Metric, symbol Device:R
- removed U3: LM556, Package_SO:SO-14_3.9x8.65mm_P1.27mm, symbol Timer:LM556
- removed U5, U6: MIC7300, digikey-footprints:SOT-753, symbol Digikey:AD8605ARTZ-REEL7
- added C16, C17, C18, C19, C20, C21, C22, C25: 100n, Capacitor_SMD:C_0402_1005Metric, symbol Device:C
- added C23, C24: 15p, Capacitor_SMD:C_0402_1005Metric, symbol Device:C
- added D1: D, Diode_SMD:D_SOD-123, symbol Device:D
- added J3: Conn_01x02, Connector_PinHeader_2.54mm:PinHeader_1x02_P2.54mm_Vertical, symbol Connector_Generic:Conn_01x02
- added J5: USB, custom:GCT_USB4105-GF-A, symbol custom:USB4105-GF-A
- added TP7: +3V3, TestPoint:TestPoint_Pad_D1.0mm, symbol Connector:TestPoint
- added TP8: +1V1, TestPoint:TestPoint_Pad_D1.0mm, symbol Connector:TestPoint
- added U3: RP2040, Package_DFN_QFN:QFN-56-1EP_7x7mm_P0.4mm_EP3.2x3.2mm, symbol MCU_RaspberryPi:RP2040
- added U5: ADP7142AUJZ-3.3, Package_TO_SOT_SMD:TSOT-23-5, symbol Regulator_Linear:ADP7142AUJZ-3.3
- added U6: W25Q40CLSNIG, footprints:WIN_SN-8_WIN, symbol custom:W25Q40CLSNIG
- added Y1: ABM8-272-T3, Crystal:Crystal_SMD_3225-4Pin_3.2x2.5mm, symbol Device:Crystal_GND24
- C11, C13: value 10u -> 1u; footprint Capacitor_SMD:C_0805_2012Metric -> Capacitor_SMD:C_0402_1005Metric
- C14, C15: value 1n -> 100n; footprint Capacitor_SMD:C_0805_2012Metric -> Capacitor_SMD:C_0402_1005Metric
- C8: value 10n -> 10u
- R10: value 500 -> 1k; footprint Resistor_SMD:R_0805_2012Metric -> Resistor_SMD:R_0402_1005Metric
- R12: value 500 -> 1k
- R13: value 8.2k -> 10k
- R2: value 42.3k -> ~
- R4: value 5k -> ~
- R6: value 10k -> ~; footprint Resistor_SMD:R_0805_2012Metric -> Resistor_SMD:R_0402_1005Metric
- R8: value 100 -> ~; footprint Resistor_SMD:R_0805_2012Metric -> Resistor_SMD:R_0402_1005Metric
- TP1: value +12 -> +6
Connections:
- net A is gone; now on net +3.3V: C14.1
- net GND: now also C16.2, C17.2, C18.2, C19.2, C20.2, C21.2, C22.2, C23.2, C24.2, C25.2, J3.2 (Pin_2), J5.A1_B12 (GND), J5.B1_A12 (GND__1), J5.SH1 (SHELL_GND), J5.SH2 (SHELL_GND__1), J5.SH3 (SHELL_GND__2), J5.SH4 (SHELL_GND__3), U3.19 (TESTEN), U3.57 (GND), U5.2 (GND), U6.4 (GND), Y1.2, Y1.4
- net PWM_A: now also U3.2 (GPIO0)
- net PWM_B: now also U3.3 (GPIO1)
- net at R6.2: now also U3.47 (USB_DP); no longer R8.1
- net +3.3V: now reaches C8.1
- net +3.3V: now also C13.1, C15.1, R13.1, C16.1, C17.1, C18.1, C19.1, C20.1, C25.1, TP7.1, U3.1 (IOVDD), U3.10 (IOVDD), U3.22 (IOVDD), U3.33 (IOVDD), U3.42 (IOVDD), U3.43 (ADC_AVDD), U3.44 (VREG_IN), U3.48 (USB_VDD), U3.49 (IOVDD), U5.4 (SENSE/ADJ), U5.5 (VOUT), U6.8 (VCC)
- net at R10.2: now also C24.1, Y1.3; no longer R12.1
- net QSPI_SS: now reaches R13.2
- net QSPI_SS: now also R12.1, U3.56 (QSPI_SS), U6.1 (*CS)
- net ~{USB_BOOT}: now reaches R12.2
- net ~{USB_BOOT}: now also J3.1 (Pin_1); no longer C13.1
- net +12V renamed +6V
- net +6V: now also D1.1 (K), U5.1 (VIN), U5.3 (EN); no longer R13.1, R6.1, U2.4 (EN)
- net B: no longer names the net of R8.2
- net B: now also U3.46 (USB_DM); no longer C11.1
- net PULSE_START renamed XOUT
- net XOUT: now also U3.21 (XOUT)
- new net: D1.2 (A), J5.A4_B9 (VBUS)
- new net +1V1: C11.1, C21.1, C22.1, TP8.1, U3.23 (DVDD), U3.45 (VREG_VOUT), U3.50 (DVDD)
- new net HV_EN: U2.4 (EN), U3.15 (GPIO12)
- new net QSPI_SCLK: U3.52 (QSPI_SCLK), U6.6 (CLK)
- new net QSPI_SD0: U3.53 (QSPI_SD0), U6.5 (DI(IO0))
- new net QSPI_SD1: U3.55 (QSPI_SD1), U6.2 (DO(IO1))
- new net QSPI_SD2: U3.54 (QSPI_SD2), U6.3 (*WP)
- new net QSPI_SD3: U3.51 (QSPI_SD3), U6.7 (*HOLD)
- new net USB_D+: J5.A6 (DP1), R6.1
- new net USB_D-: J5.A7 (DN1), R8.1
- new net XIN: C23.1, U3.20 (XIN), Y1.1
Other:
- note added: "+6 source"
- note added: "Crystal"
- note removed: "+12 source"
- note removed: "Chirp generator"
- note removed: "pulse control"
- moved on the sheet: C10, C9, J2, Q1, Q2, Q3, Q4
